File: schakelingen/Sirene/sirene/sirene.sch (KiCad schematic (older format))
At the start: 20 parts, among them Q1 BC557, Q2 BC547, Q3 BC557, Q4 BC557, Q5 TIP42

Commit message: Readme. 9V batterij in bibliotheek. Knipperlicht toegevoegd.
Parts:
- BT1: footprint Connector_PinHeader_2.54mm:PinHeader_1x02_P2.54mm_Vertical -> 9v batterij:9v batterij
Changed lines of the file:
@@
 EESchema Schematic File Version 4
-LIBS:sirene-cache
 EELAYER 30 0
 EELAYER END
@@
 F 0 "BT1" H 3718 3346 50  0000 L CNN
 F 1 "9V" H 3718 3255 50  0000 L CNN
-F 2 "Connector_PinHeader_2.54mm:PinHeader_1x02_P2.54mm_Vertical" V 3600 3310 50  0001 C CNN
+F 2 "9v batterij:9v batterij" V 3600 3310 50  0001 C CNN
 F 3 "~" V 3600 3310 50  0001 C CNN
 	1    3600 3250
